Commit message: base_refine-add_claw

File: catkin_ws/src/embodied_robot_demo/urdf/embodied_robot.urdf.xacro (robot description, xacro)
@@ -107,5 +107,5 @@
   <joint name="arm_joint_1" type="revolute">
     <parent link="arm_base_link"/><child link="arm_link_1"/>
-    <origin xyz="0 0 0.06"/><axis xyz="0 1 0"/>
+    <origin xyz="0 0 0.04"/><axis xyz="0 1 0"/>
     <limit lower="-1.20" upper="1.20" effort="35" velocity="1.5"/>
     <dynamics damping="0.8" friction="0.1"/>
@@ -127,13 +127,39 @@
   </joint>
   <link name="tool_link">
-    <visual><geometry><sphere radius="0.055"/></geometry><material name="silver"/></visual>
-    <collision><geometry><sphere radius="0.055"/></geometry></collision>
-    <inertial>
-      <mass value="0.2"/>
-      <inertia ixx="0.00024" ixy="0" ixz="0" iyy="0.00024" iyz="0" izz="0.00024"/>
+    <visual name="gripper_palm_visual">
+      <origin xyz="0 0 0.025"/>
+      <geometry><box size="0.10 0.16 0.05"/></geometry>
+      <material name="silver"/>
+    </visual>
+    <visual name="left_finger_visual">
+      <origin xyz="0 0.065 0.11"/>
+      <geometry><box size="0.04 0.03 0.14"/></geometry>
+      <material name="dark"/>
+    </visual>
+    <visual name="right_finger_visual">
+      <origin xyz="0 -0.065 0.11"/>
+      <geometry><box size="0.04 0.03 0.14"/></geometry>
+      <material name="dark"/>
+    </visual>
+    <collision name="gripper_palm_collision">
+      <origin xyz="0 0 0.025"/>
+      <geometry><box size="0.10 0.16 0.05"/></geometry>
+    </collision>
+    <collision name="left_finger_collision">
+      <origin xyz="0 0.065 0.11"/>
+      <geometry><box size="0.04 0.03 0.14"/></geometry>
+    </collision>
+    <collision name="right_finger_collision">
+      <origin xyz="0 -0.065 0.11"/>
+      <geometry><box size="0.04 0.03 0.14"/></geometry>
+    </collision>
+    <inertial>
+      <origin xyz="0 0 0.07"/>
+      <mass value="0.35"/>
+      <inertia ixx="0.00120" ixy="0" ixz="0" iyy="0.00065" iyz="0" izz="0.00125"/>
     </inertial>
   </link>
   <joint name="tool_joint" type="fixed">
-    <parent link="arm_link_2"/><child link="tool_link"/><origin xyz="0 0 0.32"/>
+    <parent link="arm_link_2"/><child link="tool_link"/><origin xyz="0 0 0.30"/>
   </joint>
   <link name="camera_link">

File: isaacgym_demo/assets/embodied_robot.urdf (robot description, URDF)
Before this commit: robot embodied_robot, 11 links, 10 joints
Links:
- link tool_link: mass 0.2 -> 0.35; geometry collision box size=0.04 0.03 0.14; collision box size=0.04 0.03 0.14
Joints:
- joint arm_joint_1: origin xyz=0 0 0.06 -> xyz=0 0 0.04
- joint tool_joint: origin xyz=0 0 0.32 -> xyz=0 0 0.30

Commit message: wheel

File: catkin_ws/src/embodied_robot_demo/urdf/embodied_robot.urdf.xacro (robot description, xacro)
@@ -5,4 +5,5 @@
   <xacro:property name="wheel_width" value="0.045"/>
   <xacro:property name="wheel_y" value="0.22"/>
+  <xacro:property name="wheel_x" value="0.18"/>
   <xacro:macro name="box_inertial" params="mass x y z">
     <inertial>
@@ -48,5 +49,5 @@
     <xacro:box_inertial mass="12.0" x="0.52" y="0.42" z="0.18"/>
   </link>
-  <xacro:macro name="wheel" params="prefix y">
+  <xacro:macro name="wheel" params="prefix x y">
     <link name="${prefix}_wheel_link">
       <visual>
@@ -64,5 +65,5 @@
       <parent link="base_link"/>
       <child link="${prefix}_wheel_link"/>
-      <origin xyz="0 ${y} -0.105"/>
+      <origin xyz="${x} ${y} -0.105"/>
       <axis xyz="0 1 0"/>
       <dynamics damping="0.05" friction="0.0"/>
@@ -72,19 +73,9 @@
     </gazebo>
   </xacro:macro>
-  <xacro:wheel prefix="left" y="${wheel_y}"/>
-  <xacro:wheel prefix="right" y="${-wheel_y}"/>
-  <link name="caster_link">
-    <visual><geometry><sphere radius="0.045"/></geometry><material name="dark"/></visual>
-    <collision><geometry><sphere radius="0.045"/></geometry></collision>
-    <inertial>
-      <mass value="0.15"/>
-      <inertia ixx="0.00012" ixy="0" ixz="0" iyy="0.00012" iyz="0" izz="0.00012"/>
-    </inertial>
-  </link>
-  <joint name="caster_joint" type="fixed">
-    <parent link="base_link"/><child link="caster_link"/>
-    <origin xyz="-0.19 0 -0.135"/>
-  </joint>
-  <gazebo reference="caster_link"><mu1>0.01</mu1><mu2>0.01</mu2></gazebo>
+  <!-- Keep the original joint names for the front wheels so existing checks remain valid. -->
+  <xacro:wheel prefix="left" x="${wheel_x}" y="${wheel_y}"/>
+  <xacro:wheel prefix="right" x="${wheel_x}" y="${-wheel_y}"/>
+  <xacro:wheel prefix="left_rear" x="${-wheel_x}" y="${wheel_y}"/>
+  <xacro:wheel prefix="right_rear" x="${-wheel_x}" y="${-wheel_y}"/>
   <link name="arm_base_link">
     <visual><geometry><cylinder radius="0.10" length="0.08"/></geometry><material name="silver"/></visual>
@@ -193,21 +184,19 @@
   </gazebo>
   <gazebo>
-    <plugin name="differential_drive_controller" filename="libgazebo_ros_diff_drive.so">
+    <plugin name="skid_steer_drive_controller" filename="libgazebo_ros_skid_steer_drive.so">
       <robotNamespace>/</robotNamespace>
-      <leftJoint>left_wheel_joint</leftJoint>
-      <rightJoint>right_wheel_joint</rightJoint>
+      <leftFrontJoint>left_wheel_joint</leftFrontJoint>
+      <rightFrontJoint>right_wheel_joint</rightFrontJoint>
+      <leftRearJoint>left_rear_wheel_joint</leftRearJoint>
+      <rightRearJoint>right_rear_wheel_joint</rightRearJoint>
       <wheelSeparation>${2 * wheel_y}</wheelSeparation>
       <wheelDiameter>${2 * wheel_radius}</wheelDiameter>
-      <wheelAcceleration>1.0</wheelAcceleration>
-      <wheelTorque>15</wheelTorque>
+      <torque>15</torque>
       <commandTopic>cmd_vel</commandTopic>
       <odometryTopic>odom</odometryTopic>
       <odometryFrame>odom</odometryFrame>
       <robotBaseFrame>base_footprint</robotBaseFrame>
-      <publishWheelTF>false</publishWheelTF>
-      <publishOdomTF>true</publishOdomTF>
-      <publishWheelJointState>true</publishWheelJointState>
+      <broadcastTF>true</broadcastTF>
       <updateRate>50</updateRate>
-      <legacyMode>false</legacyMode>
     </plugin>
   </gazebo>

File: isaacgym_demo/assets/embodied_robot.urdf (robot description, URDF)
Before this commit: robot embodied_robot, 11 links, 10 joints
Links:
- removed link caster_link
- added link left_rear_wheel_link, mass 0.8; collision cylinder length=0.045 radius=0.09; visual cylinder length=0.045 radius=0.09
- added link right_rear_wheel_link, mass 0.8; collision cylinder length=0.045 radius=0.09; visual cylinder length=0.045 radius=0.09
Joints:
- removed joint caster_joint
- added joint left_rear_wheel_joint: type continuous, parent base_link, child left_rear_wheel_link, origin xyz=-0.18 0.22 -0.105, axis 0 1 0
- added joint right_rear_wheel_joint: type continuous, parent base_link, child right_rear_wheel_link, origin xyz=-0.18 -0.22 -0.105, axis 0 1 0
- joint left_wheel_joint: origin xyz=0 0.22 -0.105 -> xyz=0.18 0.22 -0.105
- joint right_wheel_joint: origin xyz=0 -0.22 -0.105 -> xyz=0.18 -0.22 -0.105
